Commit message: Updated the uf850.urdf file

File: urdf/uf850.urdf (robot description, URDF)
Before this commit: robot uf850, 7 links, 6 joints
Joints:
- removed joint base-link_to_link3
- removed joint base_link_to_link4
- removed joint base_link_to_link5
- removed joint base_link_to_link6
- added joint link2_to_link3: type revolute, parent link2, child link3, origin xyz=0.39 0.0 -0.053 rpy=3.14 0.0 -1.57, axis 0 0 1, limit lower=-3.14 upper=3.14 effort=0.0 velocity=0.0
- added joint link3_to_link4: type revolute, parent link3, child link4, origin xyz=0.15 0.4 0 rpy=-1.57 0 0, axis 0 0 1, limit lower=0 upper=3.14 effort=0.0 velocity=0.0
- added joint link4_to_link5: type revolute, parent link4, child link5, origin xyz=0.0 0.0 0.0 rpy=-1.57 0 0, axis 0.0 0.0 1, limit lower=-1.57 upper=1.57 effort=0.0 velocity=0.0
- added joint link5_to_link6: type fixed, parent link5, child link6, origin xyz=0.0 0.0 0.0 rpy=1.57 0 0
- joint base_link_to_link1: axis (none) -> 0 0.0 1; limit (none) -> lower=-3.14 upper=3.14 effort=0.0 velocity=0.0; origin (none) -> xyz=0.0 0.0 0.362 rpy=0.0 0.0 0.0; type fixed -> revolute
- joint link1_to_link2: axis (none) -> 0 0.0 1; limit (none) -> lower=0 upper=1.57 effort=0.0 velocity=0.0; origin xyz=0.0 0.0 0.36 rpy=1.6 4.69 0.0 -> xyz=0.0 -0.051 0.0 rpy=1.57 -1.57 0; type fixed -> revolute

Commit message: For the sake of comparison

File: urdf/uf850.urdf (robot description, URDF)
Before this commit: robot uf850, 7 links, 6 joints
Joints:
- joint base_link_to_link1: origin xyz=0.0 0.0 0.362 rpy=0.0 0.0 0.0 -> xyz=0.0 0.0 0.35 rpy=0.0 0.0 0.0
- joint link1_to_link2: limit lower=0 upper=1.57 effort=0.0 velocity=0.0 -> lower=-3.14 upper=3.14 effort=0.0 velocity=0.0; origin xyz=0.0 -0.051 0.0 rpy=1.57 -1.57 0 -> xyz=0.0 0.0 0.0 rpy=1.57 -1.57 0.0
- joint link2_to_link3: axis 0 0 1 -> 0 0.0 1; origin xyz=0.39 0.0 -0.053 rpy=3.14 0.0 -1.57 -> xyz=0.39 0.0 0.0 rpy=0.0 3.14 1.57
- joint link3_to_link4: axis 0 0 1 -> 0 0.0 1; limit lower=0 upper=3.14 effort=0.0 velocity=0.0 -> lower=-3.14 upper=3.14 effort=0.0 velocity=0.0; origin xyz=0.15 0.4 0 rpy=-1.57 0 0 -> xyz=0.15 0.41 0.0 rpy=-1.57 0 0
- joint link4_to_link5: axis 0.0 0.0 1 -> 0 0.0 1; limit lower=-1.57 upper=1.57 effort=0.0 velocity=0.0 -> lower=-3.14 upper=3.14 effort=0.0 velocity=0.0; origin xyz=0.0 0.0 0.0 rpy=-1.57 0 0 -> xyz=0 -0.01 0.0 rpy=-1.57 0 0
- joint link5_to_link6: axis (none) -> 0 0.0 1; limit (none) -> lower=-3.14 upper=3.14 effort=0.0 velocity=0.0; origin xyz=0.0 0.0 0.0 rpy=1.57 0 0 -> xyz=0 -0.09 0.0 rpy=1.57 0 0; type fixed -> revolute
